Commit message: integrate velodyne for gazebo

File: sample_robot_description/urdf/robot/robot.urdf.xacro (robot description, xacro)
@@ -1,34 +1,38 @@
 <?xml version="1.0"?>
 <robot name="sample_robot" xmlns:xacro="http://ros.org/wiki/xacro">
-  <xacro:include filename="$(find sample_robot_description)/urdf/body/body.urdf.xacro"/>
-  <xacro:include filename="$(find sample_robot_description)/urdf/wheel/wheel.urdf.xacro"/>
-  <xacro:include filename="$(find sample_robot_description)/urdf/caster/caster.urdf.xacro"/>
-  <link name="base_footprint"/>
-  <xacro:base parent="base_footprint">
-    <origin xyz="0 0 0"/>
-  </xacro:base>
-  <xacro:wheel prefix="right" parent="base_link">
-    <origin xyz="0.1 -0.17 0.0" rpy="1.57 0 0" />
-    <axis xyz="0 0 -1" />
-  </xacro:wheel>
-  <xacro:wheel prefix="left" parent="base_link">
-    <origin xyz="0.1 0.17 0.0" rpy="-1.57 0 0" />
-    <axis xyz="0 0 1" />
-  </xacro:wheel>
-  <xacro:caster parent="base_link">
-    <origin xyz="-0.15 0 -0.05"/>
-  </xacro:caster>
-  <!-- ===========  Transmission ============ -->
-  <xacro:wheel_trans prefix="right" />
-  <xacro:wheel_trans prefix="left" />
-  <!-- =============== Gazebo =============== -->
-  <gazebo>
-    <plugin name="gazebo_ros_control" filename="libgazebo_ros_control.so">
-      <robotNamespace>sample_robot</robotNamespace>
-    </plugin>
-  </gazebo>
-  <xacro:body_gazebo/>
-  <xacro:wheel_gazebo prefix="right" />
-  <xacro:wheel_gazebo prefix="left" />
-  <xacro:caster_gazebo/>
+	<xacro:include filename="$(find sample_robot_description)/urdf/body/body.urdf.xacro"/>
+	<xacro:include filename="$(find sample_robot_description)/urdf/wheel/wheel.urdf.xacro"/>
+	<xacro:include filename="$(find sample_robot_description)/urdf/caster/caster.urdf.xacro"/>
+	<link name="base_footprint"/>
+	<xacro:base parent="base_footprint">
+		<origin xyz="0 0 0"/>
+	</xacro:base>
+	<xacro:wheel prefix="right" parent="base_link">
+		<origin xyz="0.1 -0.17 0.0" rpy="1.57 0 0" />
+		<axis xyz="0 0 -1" />
+	</xacro:wheel>
+	<xacro:wheel prefix="left" parent="base_link">
+		<origin xyz="0.1 0.17 0.0" rpy="-1.57 0 0" />
+		<axis xyz="0 0 1" />
+	</xacro:wheel>
+	<xacro:caster parent="base_link">
+		<origin xyz="-0.15 0 -0.05"/>
+	</xacro:caster>
+	<xacro:include filename="$(find velodyne_description)/urdf/VLP-16.urdf.xacro" />
+	<VLP-16 parent="base_link" name="velodyne" topic="/velodyne_points">
+		<origin xyz="0 0 0.052" rpy="0 0 0" />
+	</VLP-16>
+	<!-- ===========  Transmission ============ -->
+	<xacro:wheel_trans prefix="right" />
+	<xacro:wheel_trans prefix="left" />
+	<!-- =============== Gazebo =============== -->
+	<gazebo>
+		<plugin name="gazebo_ros_control" filename="libgazebo_ros_control.so">
+			<robotNamespace>sample_robot</robotNamespace>
+		</plugin>
+	</gazebo>
+	<xacro:body_gazebo/>
+	<xacro:wheel_gazebo prefix="right" />
+	<xacro:wheel_gazebo prefix="left" />
+	<xacro:caster_gazebo/>
 </robot>

Commit message: add two velodyne

File: sample_robot_description/urdf/robot/robot.urdf.xacro (robot description, xacro)
@@ -21,6 +21,9 @@
 	</xacro:caster>
 	<xacro:include filename="$(find velodyne_description)/urdf/VLP-16.urdf.xacro" />
-	<VLP-16 parent="base_link" name="velodyne" topic="/velodyne_points">
-		<origin xyz="0 0 0.052" rpy="0 0 0" />
+	<VLP-16 parent="base_link" name="velodyne_front" topic="/front_points_raw" gpu="true" hz="10">
+		<origin xyz="0.2 0 0.052" rpy="0 0 0" />
+	</VLP-16>
+	<VLP-16 parent="base_link" name="velodyne_back" topic="/back_points_raw" gpu="true" hz="10">
+		<origin xyz="-0.2 0 0.052" rpy="0 0 0" />
 	</VLP-16>
 	<!-- ===========  Transmission ============ -->

Commit message: hokuyoを追加

File: sample_robot_description/urdf/robot/robot.urdf.xacro (robot description, xacro)
@@ -4,4 +4,5 @@
 	<xacro:include filename="$(find sample_robot_description)/urdf/wheel/wheel.urdf.xacro"/>
 	<xacro:include filename="$(find sample_robot_description)/urdf/caster/caster.urdf.xacro"/>
+	<xacro:include filename="$(find sample_robot_description)/urdf/sensor/hokuyo.urdf.xacro"/>
 	<xacro:include filename="$(find sample_robot_description)/urdf/sensor/imu.gazebo.xacro"/>
 	<link name="base_footprint"/>
@@ -20,4 +21,6 @@
 		<origin xyz="-0.15 0 -0.05"/>
 	</xacro:caster>
+	<!-- velodyne -->
+	<!--
 	<xacro:include filename="$(find velodyne_description)/urdf/VLP-16.urdf.xacro" />
 	<VLP-16 parent="base_link" name="velodyne_front" topic="/front_points_raw" gpu="true" hz="10">
@@ -27,4 +30,9 @@
 		<origin xyz="-0.2 0 0.052" rpy="0 0 0" />
 	</VLP-16>
+	-->
+	<!-- Hokuyo -->
+	<xacro:hokuyo parent="base_link">
+		<origin xyz="0.2 0 0.07" rpy="0 0 0"/>
+	</xacro:hokuyo>
 	<!-- ===========  Transmission ============ -->
 	<xacro:wheel_trans prefix="right" />
